File: Arduino - 25 - Understanding Photoresistors and Photo Detectors/Arduino - 25 - Understanding Photoresistors and Photo Detectors.brd (EAGLE design)
At the start: 153.4 x 110.8 mm, 7 parts, among them U1 ARDUINO-UNO-R3-SHIELD

Commit message: Fixed Input
Parts:
- moved R1 2.54 mm to (108.9, 60.7)
Connections:
- removed net R1_2: R1.2, R2.1
- new net U1_A3: R1.2, R2.1, U1.A3
Changed lines of the file:
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@@
 <elements>
 <element name="R2" library="Tinkercad" library_urn="urn:adsk.eagle:library:30890021" package="RESAD1016W63L850D250B" package3d_urn="urn:adsk.eagle:package:31513020/2" value="1k" x="120.3597" y="73.3954" rot="R360" smashed="yes"/>
-<element name="R1" library="Tinkercad" library_urn="urn:adsk.eagle:library:30890021" package="GL5528" package3d_urn="urn:adsk.eagle:package:31494553/2" value="PHOTOCELL_GL5528" x="108.9297" y="58.1554" smashed="yes"/>
+<element name="R1" library="Tinkercad" library_urn="urn:adsk.eagle:library:30890021" package="GL5528" package3d_urn="urn:adsk.eagle:package:31494553/2" value="PHOTOCELL_GL5528" x="108.9297" y="60.6954" smashed="yes"/>
+<element name="U1" library="Tinkercad" library_urn="urn:adsk.eagle:library:30890021" package="ARDUINO-UNO-R3-SHIELD" package3d_urn="urn:adsk.eagle:package:32092383/4" value="ARDUINO-UNO-R3-SHIELD" x="47.885" y="29.845" rot="R270" smashed="yes"/>
+<element name="R3" library="Tinkercad" library_urn="urn:adsk.eagle:library:30890021" package="RESAD1016W63L850D250B" package3d_urn="urn:adsk.eagle:package:31513020/2" value="1k" x="102.4421" y="103.7908" rot="R180" smashed="yes"/>
 <element name="D1" library="Tinkercad" library_urn="urn:adsk.eagle:library:30890021" package="LEDRD254W60D565H860B" package3d_urn="urn:adsk.eagle:package:16378508/2" value="RED" x="108.9297" y="83.5554" rot="R360" smashed="yes">
 <attribute name="CATEGORY" value="Opto-Electronic" x="108.9297" y="83.5554" size="1.778" layer="27" display="off"/>
@@
 <attribute name="VALUE" value="LED_RED" x="108.9297" y="83.5554" size="1.778" layer="27" display="off"/>
 </element>
-<element name="R3" library="Tinkercad" library_urn="urn:adsk.eagle:library:30890021" package="RESAD1016W63L850D250B" package3d_urn="urn:adsk.eagle:package:31513020/2" value="1k" x="102.4421" y="103.7908" rot="R180" smashed="yes"/>
-<element name="U1" library="Tinkercad" library_urn="urn:adsk.eagle:library:30890021" package="ARDUINO-UNO-R3-SHIELD" package3d_urn="urn:adsk.eagle:package:32092383/4" value="ARDUINO-UNO-R3-SHIELD" x="47.885" y="29.845" rot="R270" smashed="yes"/>
 <element name="D2" library="Tinkercad" library_urn="urn:adsk.eagle:library:30890021" package="LEDRD254W60D565H860B_G" package3d_urn="urn:adsk.eagle:package:31997108/3" value="GREEN" x="147.0297" y="83.5554" rot="R360" smashed="yes">
 <attribute name="CATEGORY" value="Opto-Electronic" x="147.0297" y="83.5554" size="1.778" layer="27" display="off"/>
@@
 </elements>
 <signals>
-<signal name="R1_2">
+<signal name="U1_A3">
+<contactref element="R2" pad="1"/>
 <contactref element="R1" pad="2"/>
-<contactref element="R2" pad="1"/>
-<wire x1="110.6315" y1="58.1554" x2="115.2797" y2="73.3954" width="0" layer="19" extent="1-1"/>
+<contactref element="U1" pad="A3"/>
+<wire x1="115.2797" y1="73.3954" x2="110.6315" y2="60.6954" width="0" layer="19" extent="1-1"/>
+<wire x1="110.6315" y1="60.6954" x2="68.205" y2="5.715" width="0" layer="19" extent="1-1"/>
 </signal>
 <signal name="U1_GND">
@@
 </signal>
 <signal name="U1_5V">
+<contactref element="U1" pad="5V"/>
 <contactref element="R1" pad="1"/>
-<contactref element="U1" pad="5V"/>
-<wire x1="107.2279" y1="58.1554" x2="47.885" y2="5.715" width="0" layer="19" extent="1-1"/>
+<wire x1="47.885" y1="5.715" x2="107.2279" y2="60.6954" width="0" layer="19" extent="1-1"/>
+</signal>
+<signal name="U1_D4">
+<contactref element="R4" pad="2"/>
+<contactref element="U1" pad="D4"/>
+<wire x1="139.3813" y1="104.4525" x2="63.125" y2="53.975" width="0" layer="19" extent="1-1"/>
+</signal>
+<signal name="U1_D2">
+<contactref element="R3" pad="2"/>
+<contactref element="U1" pad="D2"/>
+<wire x1="97.3621" y1="103.7908" x2="68.205" y2="53.975" width="0" layer="19" extent="1-1"/>
 </signal>
 <signal name="D1_A">
@@
 <wire x1="107.5221" y1="103.7908" x2="107.6597" y2="83.5554" width="0" layer="19" extent="1-1"/>
 </signal>
-<signal name="U1_D2">
-<contactref element="R3" pad="2"/>
-<contactref element="U1" pad="D2"/>
-<wire x1="97.3621" y1="103.7908" x2="68.205" y2="53.975" width="0" layer="19" extent="1-1"/>
-</signal>
-<signal name="U1_D4">
-<contactref element="R4" pad="2"/>
-<contactref element="U1" pad="D4"/>
-<wire x1="139.3813" y1="104.4525" x2="63.125" y2="53.975" width="0" layer="19" extent="1-1"/>
-</signal>
 <signal name="D2_A">
